File: Vendo_main_board_ESP32/Vendo_main_board_ESP32.kicad_pcb (KiCad board)
At the start: 2 copper layers, 60 x 100 mm, 126 parts, among them J1 Screw_Terminal_01x04, J10 Screw_Terminal_01x03, J11 Screw_Terminal_01x02, J12 Screw_Terminal_01x03, J2 Barrel_Jack_MountingPin, J3 Conn_01x05_Pin, J4 Conn_01x05_Pin, J6 Screw_Terminal_01x04, J7 FTDI, J9 Conn_01x04_Pin, Q1 Q_NMOS_Depletion_GSD, Q2 Q_NMOS_Depletion_GSD, Q3 Q_NMOS_Depletion_GSD, Q4 Q_NMOS_Depletion_GSD, SW1 SW_Push, SW2 SW_Push, SW3 SW_Push, SW5 SW_Slide_DPDT, SW7 SW_Push, U1 AMS1117-3.3, U2 TPS54331D, U4 PC817, U5 TPL5010, U6 SOLA-IC SLM1302, U7 ESP32-WROOM-32, Y1 Crystal

Commit message: -added test pad on esp32 smart
-added test pads for jigg on smart board
Parts:
- added TP10: TestPoint, TestPoint:TestPoint_Pad_D2.5mm, B.Cu at (249.2, 74.6)
- added TP11: TestPoint, TestPoint:TestPoint_Pad_D2.5mm, B.Cu at (218.3, 98.6)
- added TP12: TestPoint, TestPoint:TestPoint_Pad_D2.5mm, B.Cu at (225.8, 63.8)
- added TP13: TestPoint, TestPoint:TestPoint_Pad_D2.5mm, B.Cu at (211.8, 67.0)
- added TP14: TestPoint, TestPoint:TestPoint_Pad_D1.5mm, B.Cu at (247.5, 93.5)
- added TP15: TestPoint, TestPoint:TestPoint_Pad_D1.5mm, B.Cu at (241.6, 96.9)
- added TP16: TestPoint, TestPoint:TestPoint_Pad_D2.5mm, B.Cu at (230.2, 106.7)
- added TP17: TestPoint, TestPoint:TestPoint_Pad_D2.5mm, B.Cu at (211.0, 109.6)
- added TP18: TestPoint, TestPoint:TestPoint_Pad_D2.5mm, B.Cu at (235.5, 117.0)
- added TP19: TestPoint, TestPoint:TestPoint_Pad_D2.5mm, B.Cu at (206.3, 99.2)
- added TP20: TestPoint, TestPoint:TestPoint_Pad_D2.5mm, B.Cu at (214.3, 98.7)
- added TP21: TestPoint, TestPoint:TestPoint_Pad_D2.5mm, B.Cu at (206.3, 104.7)
- added TP22: TestPoint, TestPoint:TestPoint_Pad_D2.5mm, B.Cu at (206.3, 116.0)
- added TP23: TestPoint, TestPoint:TestPoint_Pad_D2.5mm, B.Cu at (236.0, 106.8)
- added TP24: TestPoint, TestPoint:TestPoint_Pad_D2.5mm, B.Cu at (238.7, 112.1)
- added TP25: TestPoint, TestPoint:TestPoint_Pad_D2.5mm, B.Cu at (201.5, 49.0)
- added TP26: TestPoint, TestPoint:TestPoint_Pad_D2.5mm, B.Cu at (211.9, 55.9)
- added TP27: TestPoint, TestPoint:TestPoint_Pad_D2.5mm, B.Cu at (209.2, 47.8)
- added TP28: TestPoint, TestPoint:TestPoint_Pad_D1.5mm, B.Cu at (256.0, 62.0)
- added TP29: TestPoint, TestPoint:TestPoint_Pad_D1.5mm, B.Cu at (256.0, 59.3)
- added TP3: TestPoint, TestPoint:TestPoint_Pad_D2.5mm, B.Cu at (252.8, 43.6)
- added TP30: TestPoint, TestPoint:TestPoint_Pad_D2.5mm, B.Cu at (242.7, 103.7)
- added TP31: TestPoint, TestPoint:TestPoint_Pad_D2.5mm, B.Cu at (239.0, 57.2)
- added TP32: TestPoint, TestPoint:TestPoint_Pad_D2.5mm, B.Cu at (245.0, 108.8)
- added TP4: TestPoint, TestPoint:TestPoint_Pad_D2.5mm, B.Cu at (243.9, 31.2)
- added TP5: TestPoint, TestPoint:TestPoint_Pad_D2.5mm, B.Cu at (201.1, 60.4)
- added TP6: TestPoint, TestPoint:TestPoint_Pad_D2.5mm, B.Cu at (201.1, 66.6)
- added TP7: TestPoint, TestPoint:TestPoint_Pad_D2.5mm, B.Cu at (206.3, 85.3)
- added TP8: TestPoint, TestPoint:TestPoint_Pad_D2.5mm, B.Cu at (211.3, 84.1)
- added TP9: TestPoint, TestPoint:TestPoint_Pad_D2.5mm, B.Cu at (241.4, 83.2)
- R10, R20, R22, R24, R25, R27, R30: value 1K -> 1k
Routing:
- net GND: track 110.6 -> 134.8 mm
- net +5V: track 279.6 -> 288.7 mm, vias 6 -> 7
- net Net-(J10-Pin_1): track 14.0 -> 22.5 mm, vias 0 -> 1
- net AUX_2: track 44.9 -> 53.1 mm
- net AUX_1: track 43.6 -> 50.8 mm
- net Net-(BT1-+): track 22.8 -> 29.3 mm
- net ESP_SDA: track 62.8 -> 68.4 mm, vias 3 -> 4
- net I2C_CONFG: track 27.4 -> 33.0 mm
- net RLY_COM: track 57.4 -> 62.6 mm
- net ESP_RX: track 30.0 -> 35.2 mm
- net RLY_NC: track 17.5 -> 22.7 mm
- net USER_BTN: track 69.3 -> 74.2 mm
- net ESP_TX: track 29.5 -> 34.0 mm
- net +12V: track 135.2 -> 139.7 mm
- net RLY_NO: track 31.8 -> 35.9 mm
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
Commit message: -repush check for DRC passed
Parts:
- added TP33: TestPoint, TestPoint:TestPoint_Pad_D1.5mm, B.Cu at (249.6, 69.7)
Routing:
- net I2C_INT: track 87.1 -> 93.6 mm
- net GND: vias 168 -> 169
Changed lines of the file:
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@@
 		(embedded_fonts no)
 	)
+	(footprint "TestPoint:TestPoint_Pad_D1.5mm"
+		(layer "B.Cu")
+		(at 249.59 69.65)
+		(descr "SMD pad as test Point, diameter 1.5mm")
+		(tags "test point SMD pad")
+		(property "Reference" "TP33"
+			(at -2.82 -0.07 180)
+			(layer "B.SilkS")
+			(effects
+				(font
+					(size 0.7 0.7)
+					(thickness 0.15)
+				)
+				(justify mirror)
+			)
+		)
+		(property "Value" "TestPoint"
+			(at 0 -1.75 180)
+			(layer "B.Fab")
+			(effects
+				(font
+					(size 1 1)
+					(thickness 0.15)
+				)
+				(justify mirror)
+			)
+		)
+		(property "Datasheet" ""
+			(at 0 0 180)
+			(unlocked yes)
+			(layer "B.Fab")
+			(hide yes)
+			(effects
+				(font
+					(size 1.27 1.27)
+					(thickness 0.15)
+				)
+				(justify mirror)
+			)
+		)
+		(property "Description" "test point"
+			(at 0 0 180)
+			(unlocked yes)
+			(layer "B.Fab")
+			(hide yes)
+			(effects
+				(font
+					(size 1.27 1.27)
+					(thickness 0.15)
+				)
+				(justify mirror)
+			)
+		)
+		(property ki_fp_filters "Pin* Test*")
+		(sheetname "/")
+		(sheetfile "Vendo_main_board_ESP32.kicad_sch")
+		(attr exclude_from_pos_files)
+		(fp_circle
+			(center 0 0)
+			(end 0 -0.95)
+			(stroke
+				(width 0.12)
+				(type solid)
+			)
+			(fill no)
+			(layer "B.SilkS")
+		)
+		(fp_circle
+			(center 0 0)
+			(end 1.25 0)
+			(stroke
+				(width 0.05)
+				(type solid)
+			)
+			(fill no)
+			(layer "B.CrtYd")
+		)
+		(fp_text user "${REFERENCE}"
+			(at 0 1.65 180)
+			(layer "B.Fab")
+			(effects
+				(font
+					(size 1 1)
+					(thickness 0.15)
+				)
+				(justify mirror)
+			)
+		)
+		(pad "1" smd circle
+			(at 0 0)
+			(size 1.5 1.5)
+			(layers "B.Cu" "B.Mask")
+			(net 13 "I2C_INT")
+			(pinfunction "1")
+			(pintype "passive")
+		)
+		(embedded_fonts no)
+	)
 	(gr_rect
 		(start 239.858584 43.875)
@@
 	)
 	(via
+		(at 250.08 67.59)
+		(size 0.6)
+		(drill 0.3)
+		(layers "F.Cu" "B.Cu")
+		(net 11)
+	)
+	(via
 		(at 228.79 67.1)
 		(size 0.6)
@@
 	)
 	(via
+		(at 247.77 70.91)
+		(size 0.6)
+		(drill 0.3)
+		(layers "F.Cu" "B.Cu")
+		(net 11)
+	)
+	(via
 		(at 201.62 92.21)
 		(size 0.6)
@@
 	)
 	(via
-		(at 249.96 68.73)
+		(at 247.23 68.63)
 		(size 0.6)
 		(drill 0.3)
@@
 	)
 	(via
-		(at 248.45 69.86)
-		(size 0.6)
-		(drill 0.3)
-		(layers "F.Cu" "B.Cu")
-		(net 11)
-	)
-	(via
 		(at 222.32 90.35)
 		(size 0.6)
@@
 	)
 	(segment
+		(start 249.59 71.64)
+		(end 250.131 72.181)
+		(width 0.2)
+		(layer "B.Cu")
+		(net 13)
+	)
+	(segment
 		(start 233.22 88.22)
 		(end 231.659 86.659)
@@
 	)
 	(segment
+		(start 249.59 69.65)
+		(end 249.59 71.64)
+		(width 0.2)
+		(layer "B.Cu")
+		(net 13)
+	)
+	(segment
 		(start 232.444957 81.418)
 		(end 238.0278 81.418)
@@
 	)
 	(segment
+		(start 251.211 72.181)
+		(end 253.13 74.1)
+		(width 0.2)
+		(layer "B.Cu")
+		(net 13)
+	)
+	(segment
 		(start 220.62 79.75)
 		(end 213.8 72.93)
@@
 		(width 0.2)
 		(layer "B.Cu")
+		(net 13)
+	)
+	(segment
+		(start 250.131 72.181)
+		(end 251.211 72.181)
+		(width 0.2)
+		(layer "B.Cu")
