File: Vendo_main_board_ESP32/Vendo_main_board_ESP32.kicad_sch (KiCad schematic)
At the start: 106 parts, among them J1 Screw_Terminal_01x04, J10 Screw_Terminal_01x03, J11 Screw_Terminal_01x02, J12 Screw_Terminal_01x03, J2 Barrel_Jack_MountingPin, J3 Conn_01x05_Pin, J4 Conn_01x05_Pin, J6 Screw_Terminal_01x04, J7 FTDI, J9 Conn_01x04_Pin, Q1 Q_NMOS_Depletion_GSD, Q2 Q_NMOS_Depletion_GSD, Q3 Q_NMOS_Depletion_GSD, Q4 Q_NMOS_Depletion_GSD, SW1 SW_Push, SW2 SW_Push, SW3 SW_Push, SW5 SW_Slide_DPDT, SW7 SW_Push, U1 AMS1117-3.3, U2 TPS54331D, U4 PC817, U5 TPL5010, U6 SOLA-IC SLM1302, U7 ESP32-WROOM-32, Y1 Crystal

Commit message: -added test pad on esp32 smart
-added test pads for jigg on smart board
Parts:
- added TP10, TP11, TP12, TP13, TP16, TP17, TP18, TP19, TP20, TP21, TP22, TP23, TP24, TP25, TP26, TP27, TP3, TP30, TP31, TP32, TP4, TP5, TP6, TP7, TP8, TP9: TestPoint, TestPoint:TestPoint_Pad_D2.5mm, symbol Connector:TestPoint
- added TP14, TP15, TP28, TP29: TestPoint, TestPoint:TestPoint_Pad_D1.5mm, symbol Connector:TestPoint
- R10, R20, R22, R24, R25, R27, R30: value 1K -> 1k
Connections:
- net +12V: now also TP3.1
- net +3.3V: now also TP7.1
- net +5V: now also TP5.1
- net AUX_1: now also TP19.1
- net AUX_2: now also TP20.1
- net BTN_MODE_1: now also TP21.1
- net BTN_MODE_2: now also TP22.1
- net ESP_RX: now also TP15.1
- net ESP_SCL: now also TP9.1
- net ESP_SDA: now also TP10.1
- net ESP_TX: now also TP14.1
- net GND: now also TP12.1, TP31.1, TP32.1, TP4.1, TP6.1, TP8.1
- net I2C_CONFG: now also TP16.1
- net RLY_COM: now also TP26.1
- net RLY_NC: now also TP25.1
- net RLY_NO: now also TP27.1
- net SEG_CLK: now also TP28.1
- net SEG_DIO: now also TP29.1
- net USER_BTN: now also TP17.1
- net at J10.1 (Pin_1), JP7.2 (C): now also TP23.1
- net at J10.2 (Pin_2), JP8.1 (A), R22.2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: now also TP24.1
- net at BT1.1 (+), U6.8 (VCC1): now also TP11.1
- net at J1.4 (Pin_4), Q1.3 (D): now also TP18.1
- net at BZ1.2 (-), Q4.3 (D): now also TP30.1
- net at JP14.2 (B), R34.2, TP1.1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: now also TP13.1
Other:
- moved on the sheet: JP14, TP1

Commit message: -repush check for DRC passed
Parts:
- added TP33: TestPoint, TestPoint:TestPoint_Pad_D2.5mm, symbol Connector:TestPoint
Connections:
- net I2C_INT: now also TP33.1
Other:
- moved on the sheet: TP10, TP9
Changed lines of the file:
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@@
 	(wire
 		(pts
+			(xy 29.3363 305.6524) (xy 32.5587 305.6524)
+		)
+		(stroke
+			(width 0)
+			(type default)
+		)
+	)
+	(wire
+		(pts
 			(xy 508.0343 117.4685) (xy 511.8443 117.4685)
 		)
@@
 	(wire
 		(pts
-			(xy 30.0664 307.3867) (xy 33.3132 307.3867)
+			(xy 29.3363 295.8379) (xy 32.5831 295.8379)
 		)
 		(stroke
@@
 	(wire
 		(pts
-			(xy 30.0664 298.9001) (xy 33.3132 298.9001)
+			(xy 29.3363 287.3513) (xy 32.5831 287.3513)
 		)
 		(stroke
@@
 	(global_label "ESP_SDA"
 		(shape input)
-		(at 33.3132 307.3867 0)
+		(at 32.5831 295.8379 0)
 		(fields_autoplaced yes)
 		(effects
@@
 		)
 		(property "Intersheetrefs" "${INTERSHEET_REFS}"
-			(at 42.2325 307.3867 0)
+			(at 41.5024 295.8379 0)
 			(effects
 				(font
@@
 		)
 	)
+	(global_label "I2C_INT"
+		(shape input)
+		(at 32.5587 305.6524 0)
+		(fields_autoplaced yes)
+		(effects
+			(font
+				(size 1.016 1.016)
+			)
+			(justify left)
+		)
+		(property "Intersheetrefs" "${INTERSHEET_REFS}"
+			(at 40.5104 305.6524 0)
+			(effects
+				(font
+					(size 1.27 1.27)
+				)
+				(justify left)
+				(hide yes)
+			)
+		)
+	)
 	(global_label "RLY_DRV"
 		(shape output)
@@
 	(global_label "ESP_SCL"
 		(shape input)
-		(at 33.3132 298.9001 0)
+		(at 32.5831 287.3513 0)
 		(fields_autoplaced yes)
 		(effects
@@
 		)
 		(property "Intersheetrefs" "${INTERSHEET_REFS}"
-			(at 42.1841 298.9001 0)
+			(at 41.454 287.3513 0)
 			(effects
 				(font
@@
 	(symbol
 		(lib_id "Connector:TestPoint")
-		(at 30.0664 298.9001 90)
+		(at 29.3363 287.3513 90)
 		(unit 1)
 		(exclude_from_sim no)
@@
 		(fields_autoplaced yes)
 		(property "Reference" "TP9"
-			(at 26.7644 293.8201 90)
+			(at 26.0343 282.2713 90)
 			(effects
 				(font
@@
 		)
 		(property "Value" "TestPoint"
-			(at 26.7644 296.3601 90)
+			(at 26.0343 284.8113 90)
 			(effects
 				(font
@@
 		)
 		(property "Footprint" "TestPoint:TestPoint_Pad_D2.5mm"
-			(at 30.0664 293.8201 0)
+			(at 29.3363 282.2713 0)
 			(effects
 				(font
@@
 		)
 		(property "Datasheet" "~"
-			(at 30.0664 293.8201 0)
+			(at 29.3363 282.2713 0)
 			(effects
 				(font
@@
 		)
 		(property "Description" "test point"
-			(at 30.0664 298.9001 0)
+			(at 29.3363 287.3513 0)
 			(effects
 				(font
@@
 	(symbol
 		(lib_id "Connector:TestPoint")
-		(at 30.0664 307.3867 90)
+		(at 29.3363 295.8379 90)
 		(unit 1)
 		(exclude_from_sim no)
@@
 		(fields_autoplaced yes)
 		(property "Reference" "TP10"
-			(at 26.7644 302.3067 90)
+			(at 26.0343 290.7579 90)
 			(effects
 				(font
@@
 		)
 		(property "Value" "TestPoint"
-			(at 26.7644 304.8467 90)
+			(at 26.0343 293.2979 90)
 			(effects
 				(font
@@
 		)
 		(property "Footprint" "TestPoint:TestPoint_Pad_D2.5mm"
-			(at 30.0664 302.3067 0)
+			(at 29.3363 290.7579 0)
 			(effects
 				(font
@@
 		)
 		(property "Datasheet" "~"
-			(at 30.0664 302.3067 0)
+			(at 29.3363 290.7579 0)
 			(effects
 				(font
@@
 		)
 		(property "Description" "test point"
-			(at 30.0664 307.3867 0)
+			(at 29.3363 295.8379 0)
 			(effects
 				(font
@@
 					(unit 1)
 				)
+			)
+		)
+	)
+	(symbol
+		(lib_id "Connector:TestPoint")
+		(at 29.3363 305.6524 90)
+		(unit 1)
+		(exclude_from_sim no)
+		(in_bom yes)
+		(on_board yes)
+		(dnp no)
+		(fields_autoplaced yes)
+		(property "Reference" "TP33"
+			(at 26.0343 300.5724 90)
+			(effects
+				(font
+					(size 1.27 1.27)
+				)
+			)
+		)
+		(property "Value" "TestPoint"
+			(at 26.0343 303.1124 90)
+			(effects
+				(font
+					(size 1.27 1.27)
+				)
+			)
+		)
+		(property "Footprint" "TestPoint:TestPoint_Pad_D2.5mm"
+			(at 29.3363 300.5724 0)
+			(effects
+				(font
+					(size 1.27 1.27)
+				)
+				(hide yes)
+			)
+		)
+		(property "Datasheet" "~"
+			(at 29.3363 300.5724 0)
+			(effects
+				(font
+					(size 1.27 1.27)
+				)
+				(hide yes)
+			)
+		)
+		(property "Description" "test point"
+			(at 29.3363 305.6524 0)
+			(effects
+				(font
+					(size 1.27 1.27)
+				)
+				(hide yes)
+			)
+		)
+		(pin "1"
+		)
+		(instances
+			(project "Vendo_main_board_ESP32"
+				(path "/ce68e045-3b24-4b1f-b4c3-20bce3f1de80"
+					(reference "TP33")
+					(unit 1)
+				)
